File: SDT Neon Predradnik.brd (EAGLE design)
At the start: 152.4 x 30.1 mm, 44 parts, among them IC1 IR2153, T1 IRF840, T2 IRF840

Commit message: - zmena gridu
Parts:
- added PAD10, PAD14, PAD15, PAD16, PAD17, PAD9: (no value), wirepad:3,81/1,3
- added PAD18, PAD19, PAD20, PAD21, PAD22: (no value), wirepad:2,54/1,1
- moved IN_2 29.6 mm to (19.8, 49.1), turned to 146 degrees
- moved NEO_2A 28.6 mm to (117.8, 17.4), turned to 46 degrees
- moved L1_A 26.3 mm to (132.8, 40.1), turned to 36 degrees
- moved C8 26.1 mm to (13.4, 38.6), turned to 56 degrees
- moved PAD11 24.2 mm to (126.1, 49.3), turned to 36 degrees
- moved FIL_1A 22.8 mm to (17.2, 32.9), turned to 326 degrees
- moved IN_1 22.5 mm to (7.11, 27.3), turned to 146 degrees
- moved FIL_1B 22.1 mm to (25.0, 44.5), turned to 326 degrees
- moved PAD12 21.1 mm to (122.0, 46.4), turned to 36 degrees
- moved L1_B 20.8 mm to (124.6, 34.1), turned to 216 degrees
- moved NEO_2B 20.0 mm to (125.3, 19.9), turned to 316 degrees
- moved PAD13 18.0 mm to (117.9, 43.4), turned to 36 degrees
- moved FIL_2A 17.1 mm to (25.6, 27.2), turned to 326 degrees
- moved C7 16.2 mm to (114.6, 33.7), turned to 121 degrees
- moved FIL_2B 16.2 mm to (33.5, 38.8), turned to 326 degrees
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Routing:
- net N$14: track 174.7 -> 116.7 mm
- net N$18: track 22.4 -> 3.81 mm
- net N$7: track 116.3 -> 108.1 mm
- net N$4: track 9.72 -> 16.8 mm
- net N$9: track 21.4 -> 15.2 mm
- net N$13: track 51.4 -> 46.1 mm
- net N$3: track 16.5 -> 12.1 mm
- net N$6: track 27.7 -> 23.5 mm
- net N$5: track 31.1 -> 28.2 mm
- net N$15: track 18.6 -> 20.4 mm
- net N$17: track 5.61 -> 4.06 mm
- net N$16: track 14.6 -> 15.7 mm
- net N$8: track 5.61 -> 4.73 mm
- net N$1: track 5.08 -> 4.44 mm
- net N$19: track 20.2 -> 20.8 mm
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Other:
- board size 152.4 x 30.1 mm -> 218.5 x 218.5 mm
- board text added: "SDT"

Commit message: - final
Parts:
- added PAD23, PAD24, PAD25, PAD26: (no value), wirepad:2,54/1,1
- moved PAD17 102.0 mm to (17.8, 50.2)
- moved PAD16 72.0 mm to (3.81, 29.8)
- moved PAD18 32.2 mm to (123.2, 47.0)
- moved PAD19 29.2 mm to (118.7, 44.5)
- moved PAD9 4.58 mm to (115.6, 14.0)
- moved NEO_2A 4.07 mm to (115.2, 14.3)
- moved PAD14 4.07 mm to (132.7, 35.6)
- moved PAD20 4.02 mm to (129.5, 38.1)
- moved PAD10 3.86 mm to (137.2, 28.6)
- moved NEO_1A 3.73 mm to (132.4, 35.5), turned to 226 degrees
- moved PAD12 3.70 mm to (118.8, 44.5)
- moved PAD13 3.70 mm to (114.7, 41.5)
- moved L1_A 3.70 mm to (129.6, 38.2)
- moved PAD11 3.70 mm to (122.9, 47.4)
- moved PAD21 3.70 mm to (121.3, 32.4)
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Connections:
- new net N$20: PAD12.1, PAD13.1
- net N$8: now also PAD11.1
Routing:
- net N$8: track 4.73 -> 29.7 mm
- net N$20: track 0.00 -> 5.08 mm
- net N$5: track 28.2 -> 31.6 mm
- net N$2: track 20.1 -> 23.2 mm
- net N$14: track 116.7 -> 113.8 mm
- net N$13: track 46.1 -> 43.5 mm
- net N$7: track 108.1 -> 105.7 mm
- net N$3: track 12.1 -> 14.3 mm
- net N$1: track 4.44 -> 6.40 mm
- net N$19: track 20.8 -> 22.4 mm
- net N$4: track 16.8 -> 18.2 mm
- net N$17: track 4.06 -> 3.47 mm
Other:
- outline, holes or cut-outs redrawn
