File: SDT Neon Predradnik.sch (EAGLE design)
At the start: 44 parts, among them IC1 IR2153, T1 IRF840, T2 IRF840

Commit message: - zmena gridu
Parts:
- added PAD10, PAD14, PAD15, PAD16, PAD17, PAD9: (no value), wirepad:3,81/1,3
- added PAD18, PAD19, PAD20, PAD21, PAD22: (no value), wirepad:2,54/1,1
Changed lines of the file:
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@@
 <part name="D5" library="#PaJa_16" deviceset="1N4007" device="_10"/>
 <part name="F1" library="fuse" deviceset="FUSE" device="TE5" value="2A"/>
+<part name="PAD9" library="wirepad" deviceset="3,81/1,3" device=""/>
+<part name="PAD10" library="wirepad" deviceset="3,81/1,3" device=""/>
+<part name="PAD14" library="wirepad" deviceset="3,81/1,3" device=""/>
+<part name="PAD15" library="wirepad" deviceset="3,81/1,3" device=""/>
+<part name="PAD16" library="wirepad" deviceset="3,81/1,3" device=""/>
+<part name="PAD17" library="wirepad" deviceset="3,81/1,3" device=""/>
+<part name="PAD18" library="wirepad" deviceset="2,54/1,1" device=""/>
+<part name="PAD19" library="wirepad" deviceset="2,54/1,1" device=""/>
+<part name="PAD20" library="wirepad" deviceset="2,54/1,1" device=""/>
+<part name="PAD21" library="wirepad" deviceset="2,54/1,1" device=""/>
+<part name="PAD22" library="wirepad" deviceset="2,54/1,1" device=""/>
 </parts>
 <sheets>
@@
 <instance part="D5" gate="D" x="73.66" y="25.4" rot="R90"/>
 <instance part="F1" gate="G$1" x="17.78" y="48.26"/>
+<instance part="PAD9" gate="1" x="134.62" y="2.54" rot="R90"/>
+<instance part="PAD10" gate="1" x="139.7" y="2.54" rot="R90"/>
+<instance part="PAD14" gate="1" x="144.78" y="2.54" rot="R90"/>
+<instance part="PAD15" gate="1" x="149.86" y="2.54" rot="R90"/>
+<instance part="PAD16" gate="1" x="154.94" y="2.54" rot="R90"/>
+<instance part="PAD17" gate="1" x="160.02" y="2.54" rot="R90"/>
+<instance part="PAD18" gate="1" x="177.8" y="5.08"/>
+<instance part="PAD19" gate="1" x="182.88" y="5.08"/>
+<instance part="PAD20" gate="1" x="190.5" y="5.08"/>
+<instance part="PAD21" gate="1" x="177.8" y="2.54"/>
+<instance part="PAD22" gate="1" x="185.42" y="2.54"/>
 </instances>
 <busses>

Commit message: - final
Parts:
- added PAD23, PAD24, PAD25, PAD26: (no value), wirepad:2,54/1,1
Connections:
- new net N$20: PAD12.1, PAD13.1
- net N$8: now also PAD11.1
Changed lines of the file:
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@@
 <part name="PAD21" library="wirepad" deviceset="2,54/1,1" device=""/>
 <part name="PAD22" library="wirepad" deviceset="2,54/1,1" device=""/>
+<part name="PAD23" library="wirepad" deviceset="2,54/1,1" device=""/>
+<part name="PAD24" library="wirepad" deviceset="2,54/1,1" device=""/>
+<part name="PAD25" library="wirepad" deviceset="2,54/1,1" device=""/>
+<part name="PAD26" library="wirepad" deviceset="2,54/1,1" device=""/>
 </parts>
 <sheets>
@@
 <instance part="PAD21" gate="1" x="177.8" y="2.54"/>
 <instance part="PAD22" gate="1" x="185.42" y="2.54"/>
+<instance part="PAD23" gate="1" x="104.14" y="5.08"/>
+<instance part="PAD24" gate="1" x="99.06" y="5.08"/>
+<instance part="PAD25" gate="1" x="99.06" y="2.54"/>
+<instance part="PAD26" gate="1" x="104.14" y="2.54"/>
 </instances>
 <busses>
@@
 <pinref part="NEO_1B" gate="G$1" pin="1"/>
 <wire x1="208.28" y1="25.4" x2="203.2" y2="25.4" width="0.1524" layer="91"/>
+<pinref part="PAD11" gate="G$1" pin="1"/>
+<wire x1="198.12" y1="43.18" x2="208.28" y2="43.18" width="0.1524" layer="91"/>
+<wire x1="208.28" y1="43.18" x2="208.28" y2="27.94" width="0.1524" layer="91"/>
 </segment>
 </net>
@@
 </segment>
 </net>
+<net name="N$20" class="0">
+<segment>
+<pinref part="PAD12" gate="G$1" pin="1"/>
+<pinref part="PAD13" gate="G$1" pin="1"/>
+<wire x1="198.12" y1="40.64" x2="198.12" y2="38.1" width="0.1524" layer="91"/>
+</segment>
+</net>
